File: MARIA/cd40/cd40.kicad_sch (KiCad schematic)
At the start: 2 parts

Commit message: CHECK KICAD
Connections:
- net VEE: no longer U?.7 (VEE)
- new net GND: U?.7 (VEE)
Changed lines of the file:
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@@
+    )
+  )
+  (global_label "GND" (shape input) (at 130.81 104.14 270) (fields_autoplaced)
+    (effects (font (size 1.27 1.27)) (justify right))
+    (property "Intersheet References" "${INTERSHEET_REFS}" (id 0) (at 130.8894 110.4236 90)
+      (effects (font (size 1.27 1.27)) (justify right) hide)
     )
   )
@@
     )
     (property "Datasheet" "" (id 3) (at 135.89 64.77 0)
-      (effects (font (size 1.27 1.27)) hide)
-    )
-    (pin "1")
-  )
-  (symbol (lib_id "power:VEE") (at 130.81 104.14 180) (unit 1)
-    (in_bom yes) (on_board yes) (fields_autoplaced)
-    (property "Reference" "#PWR?" (id 0) (at 130.81 100.33 0)
-      (effects (font (size 1.27 1.27)) hide)
-    )
-    (property "Value" "VEE" (id 1) (at 130.81 109.22 0))
-    (property "Footprint" "" (id 2) (at 130.81 104.14 0)
-      (effects (font (size 1.27 1.27)) hide)
-    )
-    (property "Datasheet" "" (id 3) (at 130.81 104.14 0)
       (effects (font (size 1.27 1.27)) hide)
     )
@@
       (reference "#PWR?") (unit 1) (value "VDD") (footprint "")
     )
-    (path "/ad4a0cfd-1d37-466a-b358-2e8c63e846b7"
-      (reference "#PWR?") (unit 1) (value "VEE") (footprint "")
-    )
     (path "/ae7c0ed9-c5ba-4a47-8c40-3d33da00c4b1"
