File: MARIA/SCHMATIC/cd40.kicad_sch (KiCad schematic)
At the start: 11 parts

Commit message: I/O NAMES CHANGE
Connections:
- net I/O 0: no longer U?.13 (X0)
- net I/O 1: no longer U?.14 (X1)
- net I/O 2: no longer U?.15 (X2)
- net I/O 3: no longer U?.12 (X3)
- net I/O 4: no longer U?.1 (X4)
- net I/O 5: no longer U?.5 (X5)
- net I/O 6: no longer U?.2 (X6)
- net I/O 7: no longer U?.4 (X7)
- new net I/O 10: U?.15 (X2)
- new net I/O 11: U?.12 (X3)
- new net I/O 12: U?.1 (X4)
- new net I/O 13: U?.5 (X5)
- new net I/O 14: U?.2 (X6)
- new net I/O 15: U?.4 (X7)
- new net I/O 8: U?.13 (X0)
- new net I/O 9: U?.14 (X1)
Changed lines of the file:
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@@
     )
   )
-  (global_label "I{slash}O 5" (shape input) (at 267.97 137.16 0) (fields_autoplaced)
-    (effects (font (size 1.27 1.27)) (justify left))
-    (property "Intersheet References" "${INTERSHEET_REFS}" (id 0) (at 275.826 137.0806 0)
+  (global_label "I{slash}O 13" (shape input) (at 267.97 137.16 0) (fields_autoplaced)
+    (effects (font (size 1.27 1.27)) (justify left))
+    (property "Intersheet References" "${INTERSHEET_REFS}" (id 0) (at 277.0355 137.0806 0)
       (effects (font (size 1.27 1.27)) (justify left) hide)
     )
@@
     )
   )
-  (global_label "I{slash}O 6" (shape input) (at 260.35 139.7 0) (fields_autoplaced)
-    (effects (font (size 1.27 1.27)) (justify left))
-    (property "Intersheet References" "${INTERSHEET_REFS}" (id 0) (at 268.206 139.6206 0)
+  (global_label "I{slash}O 14" (shape input) (at 260.35 139.7 0) (fields_autoplaced)
+    (effects (font (size 1.27 1.27)) (justify left))
+    (property "Intersheet References" "${INTERSHEET_REFS}" (id 0) (at 269.4155 139.6206 0)
       (effects (font (size 1.27 1.27)) (justify left) hide)
     )
@@
     )
   )
-  (global_label "I{slash}O 7" (shape input) (at 267.97 142.24 0) (fields_autoplaced)
-    (effects (font (size 1.27 1.27)) (justify left))
-    (property "Intersheet References" "${INTERSHEET_REFS}" (id 0) (at 275.826 142.1606 0)
+  (global_label "I{slash}O 15" (shape input) (at 267.97 142.24 0) (fields_autoplaced)
+    (effects (font (size 1.27 1.27)) (justify left))
+    (property "Intersheet References" "${INTERSHEET_REFS}" (id 0) (at 277.0355 142.1606 0)
       (effects (font (size 1.27 1.27)) (justify left) hide)
     )
@@
     )
   )
-  (global_label "I{slash}O 1" (shape input) (at 267.97 127 0) (fields_autoplaced)
+  (global_label "I{slash}O 9" (shape input) (at 267.97 127 0) (fields_autoplaced)
     (effects (font (size 1.27 1.27)) (justify left))
     (property "Intersheet References" "${INTERSHEET_REFS}" (id 0) (at 275.826 126.9206 0)
@@
     )
   )
-  (global_label "I{slash}O 4" (shape input) (at 260.35 134.62 0) (fields_autoplaced)
-    (effects (font (size 1.27 1.27)) (justify left))
-    (property "Intersheet References" "${INTERSHEET_REFS}" (id 0) (at 268.206 134.5406 0)
+  (global_label "I{slash}O 12" (shape input) (at 260.35 134.62 0) (fields_autoplaced)
+    (effects (font (size 1.27 1.27)) (justify left))
+    (property "Intersheet References" "${INTERSHEET_REFS}" (id 0) (at 269.4155 134.5406 0)
       (effects (font (size 1.27 1.27)) (justify left) hide)
     )
@@
     )
   )
-  (global_label "I{slash}O 3" (shape input) (at 267.97 132.08 0) (fields_autoplaced)
-    (effects (font (size 1.27 1.27)) (justify left))
-    (property "Intersheet References" "${INTERSHEET_REFS}" (id 0) (at 275.826 132.0006 0)
+  (global_label "I{slash}O 11" (shape input) (at 267.97 132.08 0) (fields_autoplaced)
+    (effects (font (size 1.27 1.27)) (justify left))
+    (property "Intersheet References" "${INTERSHEET_REFS}" (id 0) (at 277.0355 132.0006 0)
       (effects (font (size 1.27 1.27)) (justify left) hide)
     )
@@
     )
   )
-  (global_label "I{slash}O 0" (shape input) (at 260.35 124.46 0) (fields_autoplaced)
+  (global_label "I{slash}O 8" (shape input) (at 260.35 124.46 0) (fields_autoplaced)
     (effects (font (size 1.27 1.27)) (justify left))
     (property "Intersheet References" "${INTERSHEET_REFS}" (id 0) (at 268.206 124.3806 0)
@@
     )
   )
-  (global_label "I{slash}O 2" (shape input) (at 260.35 129.54 0) (fields_autoplaced)
-    (effects (font (size 1.27 1.27)) (justify left))
-    (property "Intersheet References" "${INTERSHEET_REFS}" (id 0) (at 268.206 129.4606 0)
-      (effects (font (size 1.27 1.27)) (justify left) hide)
-    )
+  (global_label "I{slash}O 10" (shape input) (at 260.35 129.54 0) (fields_autoplaced)
+    (effects (font (size 1.27 1.27)) (justify left))
+    (property "Intersheet References" "${INTERSHEET_REFS}" (id 0) (at 269.4155 129.4606 0)
+      (effects (font (size 1.27 1.27)) (justify left) hide)
+    )

Commit message: HEADINGS
Other:
- note added: "1ST MULTIPLEXER"
- note added: "2ND MULTIPLEXER"
- note added: "ESP8266 BOOTING CIRCUIT"
- moved on the sheet: U?
