File: USAID/bot circuit design (1).kicad_sch (KiCad schematic)
At the start: 14 parts, among them M1 Motor_DC, M2 Motor_DC, SW1 FLASH, SW2 RESET, U1 AMS1117-3.3V

Commit message: CORRECT ERRORS
FTDI CONNECTION FIXED  INTERFACE BOARD CONNECTION CHECK
Connections:
- net FTDI RX: now also U?.22 (GPIO1/TXD); no longer U?.21 (GPIO3/RXD)
- net FTDI TX: now also U?.21 (GPIO3/RXD); no longer U?.22 (GPIO1/TXD)
Changed lines of the file:
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@@
     )
   )
-  (global_label "FTDI RX" (shape input) (at 95.25 71.12 0) (fields_autoplaced)
+  (global_label "FTDI TX" (shape input) (at 95.25 71.12 0) (fields_autoplaced)
     (effects (font (size 1.27 1.27)) (justify left))
-    (property "Intersheet References" "${INTERSHEET_REFS}" (id 0) (at 105.0412 71.0406 0)
+    (property "Intersheet References" "${INTERSHEET_REFS}" (id 0) (at 104.7388 71.0406 0)
       (effects (font (size 1.27 1.27)) (justify left) hide)
     )
@@
     )
   )
-  (global_label "FTDI TX" (shape input) (at 95.25 66.04 0) (fields_autoplaced)
+  (global_label "FTDI RX" (shape input) (at 95.25 66.04 0) (fields_autoplaced)
     (effects (font (size 1.27 1.27)) (justify left))
-    (property "Intersheet References" "${INTERSHEET_REFS}" (id 0) (at 104.7388 65.9606 0)
+    (property "Intersheet References" "${INTERSHEET_REFS}" (id 0) (at 105.0412 65.9606 0)
       (effects (font (size 1.27 1.27)) (justify left) hide)
     )
