File: USAID/bot sch and pcb.kicad_pcb (KiCad board)
At the start: 2 copper layers, 61 x 48.3 mm, 14 parts, among them J1 FTDI, M1 Motor_DC, M2 Motor_DC, SW1 RESET, SW2 FLASH, U1 ESP-12E, U2 L293D, U3 AMS1117-3.3V

Commit message: filler added
Routing:
- added copper zone on F.Cu, net GND
Other:
- board size 61 x 48.3 mm -> 61 x 45.7 mm
Changed lines of the file:
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@@
     )
   )
-  (gr_rect (start 152.4 40.64) (end 213.36 88.9) (layer "Edge.Cuts") (width 0.1) (fill none))
+  (gr_line (start 152.4 91.44) (end 152.4 45.72) (layer "Edge.Cuts") (width 0.1))
+  (gr_line (start 177.8 48.26) (end 198.12 48.26) (layer "Edge.Cuts") (width 0.1))
+  (gr_line (start 198.12 45.72) (end 213.36 45.72) (layer "Edge.Cuts") (width 0.1))
+  (gr_line (start 213.36 91.44) (end 152.4 91.44) (layer "Edge.Cuts") (width 0.1))
+  (gr_line (start 177.8 45.72) (end 177.8 48.26) (layer "Edge.Cuts") (width 0.1))
+  (gr_line (start 152.4 45.72) (end 177.8 45.72) (layer "Edge.Cuts") (width 0.1))
+  (gr_line (start 198.12 48.26) (end 198.12 45.72) (layer "Edge.Cuts") (width 0.1))
+  (gr_line (start 213.36 45.72) (end 213.36 91.44) (layer "Edge.Cuts") (width 0.1))
   (gr_text "POCOBOT" (at 165.1 83.82) (layer "F.SilkS")
     (effects (font (size 2 3) (thickness 0.15)) (justify mirror))
@@
   (segment (start 195.56 56.38) (end 193.9597 56.38) (width 0.3) (layer "F.Cu") (net 29))
   (segment (start 176.2094 51.0259) (end 175.1503 52.085) (width 0.3) (layer "F.Cu") (net 29))
-  (zone (net 0) (net_name "") (layer "F.Cu") (hatch edge 0.508)
-    (connect_pads (clearance 0))
-    (min_thickness 0.254)
-    (keepout (tracks not_allowed) (vias not_allowed) (pads not_allowed ) (copperpour allowed) (footprints allowed))
-    (fill (thermal_gap 0.508) (thermal_bridge_width 0.508))
+  (zone (net 7) (net_name "GND") (layer "F.Cu") (hatch edge 0.508)
+    (connect_pads (clearance 0.508))
+    (min_thickness 0.254) (filled_areas_thickness no)
+    (fill yes (thermal_gap 0.508) (thermal_bridge_width 0.508))
     (polygon
       (pts
-        (xy 213.36 88.9)
-        (xy 152.4 88.9)
-        (xy 152.4 40.64)
-        (xy 213.36 40.64)
+        (xy 177.8 48.26)
+        (xy 198.12 48.26)
+        (xy 198.12 45.72)
+        (xy 213.36 45.72)
+        (xy 213.36 91.44)
+        (xy 152.4 91.44)
+        (xy 152.4 45.72)
+        (xy 177.8 45.72)
       )
     )
@@
   (zone (net 7) (net_name "GND") (layer "B.Cu") (hatch edge 0.508)
     (connect_pads (clearance 0.508))
-    (min_thickness 0.254)
-    (fill (thermal_gap 0.508) (thermal_bridge_width 0.508))
+    (min_thickness 0.254) (filled_areas_thickness no)
+    (fill yes (thermal_gap 0.508) (thermal_bridge_width 0.508))
     (polygon
       (pts
-        (xy 213.36 88.9)
-        (xy 152.4 88.9)
-        (xy 152.4 40.64)
-        (xy 213.36 40.64)
+        (xy 177.8 48.26)
+        (xy 198.12 48.26)
+        (xy 198.12 45.72)
+        (xy 213.36 45.72)
+        (xy 213.36 91.44)
+        (xy 152.4 91.44)
+        (xy 152.4 45.72)
+        (xy 177.8 45.72)
       )
     )
